Commit message: fix bug again

File: robots/a1_imu_description/xacro/gazebo.xacro (robot description, xacro)
@@ -18,5 +18,5 @@
         </plugin>
     </gazebo>
-    <!-- <gazebo>
+    <gazebo>
         <plugin name="p3d" filename="libgazebo_ros_p3d.so">
             <alwaysOn>true</alwaysOn>
@@ -26,5 +26,5 @@
             <frameName>world</frameName>
         </plugin>
-    </gazebo> -->
+    </gazebo>
     <!-- Show foot position  -->
     <!-- problem: p3d_FL_foot_controller and other sensors are not working, although we set bodyName be FL_foot_imu_link, it measures FL_calf
@@ -288,5 +288,5 @@
         <material>Gazebo/Red</material>
     </gazebo>
-    <gazebo reference="FL_foot_imu_link">
+    <!-- <gazebo reference="FL_foot_imu_link">
         <mu1>0.2</mu1>
         <mu2>0.2</mu2>
@@ -307,5 +307,5 @@
         <mu2>0.2</mu2>
         <material>Gazebo/Red</material>
-    </gazebo>
+    </gazebo> -->
     <!-- FL leg -->
     <gazebo reference="FL_hip">

File: robots/a1_imu_description/xacro/leg.xacro (robot description, xacro)
@@ -167,9 +167,9 @@
         </joint>
     <link name="${name}_foot_imu_link">
-        <inertial>
+        <!-- <inertial>
             <mass value="0.001"/>
             <origin rpy="0 0 0" xyz="0 0 0"/>
             <inertia ixx="0.0001" ixy="0" ixz="0" iyy="0.0001" iyz="0" izz="0.0001"/>
-        </inertial>
+        </inertial> -->
         <visual>
             <origin rpy="0 0 0" xyz="0 0 0"/>
@@ -179,5 +179,5 @@
             <material name="red"/>
         </visual>
-        <collision>
+        <!-- <collision>
             <origin rpy="0 0 0" xyz="0 0 0"/>
             <geometry>
@@ -192,5 +192,5 @@
                 </friction>
             </surface>
-        </collision>
+        </collision> -->
     </link>
     <joint name="${name}_imu_joint" type="fixed">

Commit message: fix bug: must add dynamics

File: robots/a1_imu_description/xacro/gazebo.xacro (robot description, xacro)
@@ -288,5 +288,5 @@
         <material>Gazebo/Red</material>
     </gazebo>
-    <!-- <gazebo reference="FL_foot_imu_link">
+    <gazebo reference="FL_foot_imu_link">
         <mu1>0.2</mu1>
         <mu2>0.2</mu2>
@@ -307,5 +307,5 @@
         <mu2>0.2</mu2>
         <material>Gazebo/Red</material>
-    </gazebo> -->
+    </gazebo>
     <!-- FL leg -->
     <gazebo reference="FL_hip">

File: robots/a1_imu_description/xacro/leg.xacro (robot description, xacro)
@@ -167,9 +167,9 @@
         </joint>
     <link name="${name}_foot_imu_link">
-        <!-- <inertial>
+        <inertial>
             <mass value="0.001"/>
             <origin rpy="0 0 0" xyz="0 0 0"/>
             <inertia ixx="0.0001" ixy="0" ixz="0" iyy="0.0001" iyz="0" izz="0.0001"/>
-        </inertial> -->
+        </inertial>
         <visual>
             <origin rpy="0 0 0" xyz="0 0 0"/>
@@ -179,5 +179,5 @@
             <material name="red"/>
         </visual>
-        <!-- <collision>
+        <collision>
             <origin rpy="0 0 0" xyz="0 0 0"/>
             <geometry>
@@ -192,5 +192,5 @@
                 </friction>
             </surface>
-        </collision> -->
+        </collision>
     </link>
     <joint name="${name}_imu_joint" type="fixed">
