Commit message: fix bug in a1_imu

File: robots/a1_imu_description/urdf/a1_imu.urdf (robot description, URDF)
Before this commit: robot a1_description, 23 links, 22 joints
Links:
- added link FL_foot_imu_link, mass 0.001; collision sphere radius=.0001; visual box size=0.001 0.001 0.001
- added link FR_foot_imu_link, mass 0.001; collision sphere radius=.0001; visual box size=0.001 0.001 0.001
- added link RL_foot_imu_link, mass 0.001; collision sphere radius=.0001; visual box size=0.001 0.001 0.001
- added link RR_foot_imu_link, mass 0.001; collision sphere radius=.0001; visual box size=0.001 0.001 0.001
- link FL_calf: geometry collision box size=0.2 0.016 0.016; visual mesh filename=package://a1_imu_description/meshes/calf.dae scale=1 1 1
- link FL_hip: geometry collision cylinder length=0.04 radius=0.046; visual mesh filename=package://a1_imu_description/meshes/hip.dae scale=1 1 1
- link FL_thigh: geometry collision box size=0.2 0.0245 0.034; visual mesh filename=package://a1_imu_description/meshes/thigh.dae scale=1 1 1
- link FR_calf: geometry collision box size=0.2 0.016 0.016; visual mesh filename=package://a1_imu_description/meshes/calf.dae scale=1 1 1
- link FR_hip: geometry collision cylinder length=0.04 radius=0.046; visual mesh filename=package://a1_imu_description/meshes/hip.dae scale=1 1 1
- link FR_thigh: geometry collision box size=0.2 0.0245 0.034; visual mesh filename=package://a1_imu_description/meshes/thigh_mirror.dae scale=1 1 1
- link RL_calf: geometry collision box size=0.2 0.016 0.016; visual mesh filename=package://a1_imu_description/meshes/calf.dae scale=1 1 1
- link RL_hip: geometry collision cylinder length=0.04 radius=0.046; visual mesh filename=package://a1_imu_description/meshes/hip.dae scale=1 1 1
- link RL_thigh: geometry collision box size=0.2 0.0245 0.034; visual mesh filename=package://a1_imu_description/meshes/thigh.dae scale=1 1 1
- link RR_calf: geometry collision box size=0.2 0.016 0.016; visual mesh filename=package://a1_imu_description/meshes/calf.dae scale=1 1 1
- link RR_hip: geometry collision cylinder length=0.04 radius=0.046; visual mesh filename=package://a1_imu_description/meshes/hip.dae scale=1 1 1
- link RR_thigh: geometry collision box size=0.2 0.0245 0.034; visual mesh filename=package://a1_imu_description/meshes/thigh_mirror.dae scale=1 1 1
- link trunk: geometry collision mesh filename=package://a1_imu_description/meshes/trunk.dae scale=1 1 1; visual mesh filename=package://a1_imu_description/meshes/trunk.dae scale=1 1 1
Joints:
- added joint FL_imu_joint: type fixed, parent FL_foot, child FL_foot_imu_link, origin xyz=0 0 0 rpy=0 0 0
- added joint FR_imu_joint: type fixed, parent FR_foot, child FR_foot_imu_link, origin xyz=0 0 0 rpy=0 0 0
- added joint RL_imu_joint: type fixed, parent RL_foot, child RL_foot_imu_link, origin xyz=0 0 0 rpy=0 0 0
- added joint RR_imu_joint: type fixed, parent RR_foot, child RR_foot_imu_link, origin xyz=0 0 0 rpy=0 0 0

File: robots/a1_imu_description/xacro/gazebo.xacro (robot description, xacro)
@@ -10,5 +10,5 @@
     <!-- simulate a body pose sensor -->
     <gazebo>
-        <plugin name="p3d" filename="libgazebo_ros_p3d.so">
+        <plugin name="p3d_body" filename="libgazebo_ros_p3d.so">
         <alwaysOn>true</alwaysOn>
         <updateRate>100.0</updateRate>
@@ -16,62 +16,85 @@
         <topicName>body_pose_ground_truth</topicName>
         <frameName>world</frameName>
-        <xyzOffsets>0 0 0.0</xyzOffsets>
-        <rpyOffsets>0 0 0.0</rpyOffsets>
-        </plugin>
-    </gazebo>
-    <gazebo>
+        </plugin>
+    </gazebo>
+    <!-- <gazebo>
         <plugin name="p3d" filename="libgazebo_ros_p3d.so">
-            <always_on>true</always_on>
-            <update_rate>200</update_rate>
+            <alwaysOn>true</alwaysOn>
+            <updateRate>100.0</updateRate>
             <bodyName>base</bodyName>
-            <topicName>/torso_odom</topicName>
+            <topicName>torso_odom</topicName>
             <frameName>world</frameName>
-            <xyzOffset>0 0 0</xyzOffset>
-            <rpyOffset>0 0 0</rpyOffset>
-        </plugin>
-    </gazebo>
+        </plugin>
+    </gazebo> -->
     <!-- Show foot position  -->
-    <gazebo>
-        <plugin name="p3d" filename="libgazebo_ros_p3d.so">
-            <always_on>true</always_on>
-            <update_rate>200</update_rate>
-            <bodyName>FL_foot_imu_link</bodyName>
-            <topicName>/FL_foot_odom</topicName>
+    <!-- problem: p3d_FL_foot_controller and other sensors are not working, although we set bodyName be FL_foot_imu_link, it measures FL_calf
+         solution: gazebo supress fixed joint by default, then FL_foot and FL_foot_imu_link won't show in gazebo hence p3d cannot find them
+             so we need following preserveFixedJoint settings to make sure FL_foot and FL_foot_imu_link do not get supressed  -->
+    <gazebo reference="FL_foot_fixed">
+        <disableFixedJointLumping>true</disableFixedJointLumping>
+        <preserveFixedJoint>true</preserveFixedJoint>
+    </gazebo>
+    <gazebo reference="FL_imu_joint">
+        <disableFixedJointLumping>true</disableFixedJointLumping>
+        <preserveFixedJoint>true</preserveFixedJoint>
+    </gazebo>
+    <gazebo reference="FR_foot_fixed">
+        <disableFixedJointLumping>true</disableFixedJointLumping>
+        <preserveFixedJoint>true</preserveFixedJoint>
+    </gazebo>
+    <gazebo reference="FR_imu_joint">
+        <disableFixedJointLumping>true</disableFixedJointLumping>
+        <preserveFixedJoint>true</preserveFixedJoint>
+    </gazebo>
+    <gazebo reference="RL_foot_fixed">
+        <disableFixedJointLumping>true</disableFixedJointLumping>
+        <preserveFixedJoint>true</preserveFixedJoint>
+    </gazebo>
+    <gazebo reference="RL_imu_joint">
+        <disableFixedJointLumping>true</disableFixedJointLumping>
+        <preserveFixedJoint>true</preserveFixedJoint>
+    </gazebo>
+    <gazebo reference="RR_foot_fixed">
+        <disableFixedJointLumping>true</disableFixedJointLumping>
+        <preserveFixedJoint>true</preserveFixedJoint>
+    </gazebo>
+    <gazebo reference="RR_imu_joint">
+        <disableFixedJointLumping>true</disableFixedJointLumping>
+        <preserveFixedJoint>true</preserveFixedJoint>
+    </gazebo>
+    <gazebo>
+        <plugin name="p3d_fl_foot" filename="libgazebo_ros_p3d.so">
+          <alwaysOn>true</alwaysOn>
+          <updateRate>100.0</updateRate>
+          <bodyName>FL_foot_imu_link</bodyName>
+          <topicName>FL_foot_odom</topicName>
+          <frameName>world</frameName>
+        </plugin>
+    </gazebo>
+    <gazebo>
+        <plugin name="p3d_fr_foot" filename="libgazebo_ros_p3d.so">
+            <alwaysOn>true</alwaysOn>
+            <updateRate>100.0</updateRate>
+            <bodyName>FR_foot_imu_link</bodyName>
+            <topicName>FR_foot_odom</topicName>
             <frameName>world</frameName>
-            <xyzOffset>0 0 0</xyzOffset>
-            <rpyOffset>0 0 0</rpyOffset>
-        </plugin>
-    </gazebo>
-    <gazebo>
-        <plugin name="p3d" filename="libgazebo_ros_p3d.so">
-            <always_on>true</always_on>
-            <update_rate>200</update_rate>
-            <bodyName>FR_foot_imu_link</bodyName>
-            <topicName>/FR_foot_odom</topicName>
+        </plugin>
+    </gazebo>
+    <gazebo>
+        <plugin name="p3d_rl_foot" filename="libgazebo_ros_p3d.so">
+            <alwaysOn>true</alwaysOn>
+            <updateRate>100.0</updateRate>
+            <bodyName>RL_foot_imu_link</bodyName>
+            <topicName>RL_foot_odom</topicName>
             <frameName>world</frameName>
-            <xyzOffset>0 0 0</xyzOffset>
-            <rpyOffset>0 0 0</rpyOffset>
-        </plugin>
-    </gazebo>
-    <gazebo>
-        <plugin name="p3d" filename="libgazebo_ros_p3d.so">
-            <always_on>true</always_on>
-            <update_rate>200</update_rate>
-            <bodyName>RL_foot_imu_link</bodyName>
-            <topicName>/RL_foot_odom</topicName>
+        </plugin>
+    </gazebo>
+    <gazebo>
+        <plugin name="p3d_rr_foot" filename="libgazebo_ros_p3d.so">
+            <alwaysOn>true</alwaysOn>
+            <updateRate>100.0</updateRate>
+            <bodyName>RR_foot_imu_link</bodyName>
+            <topicName>RR_foot_odom</topicName>
             <frameName>world</frameName>
-            <xyzOffset>0 0 0</xyzOffset>
-            <rpyOffset>0 0 0</rpyOffset>
-        </plugin>
-    </gazebo>
-    <gazebo>
-        <plugin name="p3d" filename="libgazebo_ros_p3d.so">
-            <always_on>true</always_on>
-            <update_rate>200</update_rate>
-            <bodyName>RR_foot_imu_link</bodyName>
-            <topicName>/RR_foot_odom</topicName>
-            <frameName>world</frameName>
-            <xyzOffset>0 0 0</xyzOffset>
-            <rpyOffset>0 0 0</rpyOffset>
         </plugin>
     </gazebo>
@@ -87,5 +110,5 @@
         <sensor name="imu_sensor" type="imu">
             <always_on>true</always_on>
-            <update_rate>400</update_rate>
+            <!-- <updateRate>400</updateRate> -->
             <visualize>true</visualize>
             <topic>__default_topic__</topic>
@@ -107,5 +130,5 @@
         <sensor name="FL_foot_imu_sensor" type="imu">
             <always_on>true</always_on>
-            <update_rate>400</update_rate>
+            <!-- <updateRate>400</updateRate> -->
             <visualize>true</visualize>
             <topic>FL_foot_imu</topic>
@@ -126,5 +149,5 @@
         <sensor name="FR_foot_imu_sensor" type="imu">
             <always_on>true</always_on>
-            <update_rate>400</update_rate>
+            <!-- <updateRate>400</updateRate> -->
             <visualize>true</visualize>
             <topic>FR_foot_imu</topic>
@@ -145,5 +168,5 @@
         <sensor name="RL_foot_imu_sensor" type="imu">
             <always_on>true</always_on>
-            <update_rate>400</update_rate>
+            <!-- <updateRate>400</updateRate> -->
             <visualize>true</visualize>
             <topic>RL_foot_imu</topic>
@@ -164,5 +187,5 @@
         <sensor name="RR_foot_imu_sensor" type="imu">
             <always_on>true</always_on>
-            <update_rate>400</update_rate>
+            <!-- <updateRate>400</updateRate> -->
             <visualize>true</visualize>
             <topic>RR_foot_imu</topic>
@@ -182,5 +205,5 @@
     <gazebo reference="FR_calf">
         <sensor name="FR_foot_contact" type="contact">
-        <update_rate>100</update_rate>
+        <!-- <updateRate>100</updateRate> -->
         <plugin name="contactPlugin" filename="libunitreeFootContactPlugin.so"/>
         <contact>
@@ -191,5 +214,5 @@
     <gazebo reference="FL_calf">
         <sensor name="FL_foot_contact" type="contact">
-        <update_rate>100</update_rate>
+        <!-- <updateRate>100</updateRate> -->
         <plugin name="contactPlugin" filename="libunitreeFootContactPlugin.so"/>
         <contact>
@@ -200,5 +223,5 @@
     <gazebo reference="RR_calf">
         <sensor name="RR_foot_contact" type="contact">
-        <update_rate>100</update_rate>
+        <!-- <updateRate>100</updateRate> -->
         <plugin name="contactPlugin" filename="libunitreeFootContactPlugin.so"/>
         <contact>
@@ -209,5 +232,5 @@
     <gazebo reference="RL_calf">
         <sensor name="RL_foot_contact" type="contact">
-        <update_rate>100</update_rate>
+        <!-- <updateRate>100</updateRate> -->
         <plugin name="contactPlugin" filename="libunitreeFootContactPlugin.so"/>
         <contact>
@@ -265,4 +288,24 @@
         <material>Gazebo/Red</material>
     </gazebo>
+    <gazebo reference="FL_foot_imu_link">
+        <mu1>0.2</mu1>
+        <mu2>0.2</mu2>
+        <material>Gazebo/Red</material>
+    </gazebo>
+    <gazebo reference="FR_foot_imu_link">
+        <mu1>0.2</mu1>
+        <mu2>0.2</mu2>
+        <material>Gazebo/Red</material>
+    </gazebo>
+    <gazebo reference="RL_foot_imu_link">
+        <mu1>0.2</mu1>
+        <mu2>0.2</mu2>
+        <material>Gazebo/Red</material>
+    </gazebo>
+    <gazebo reference="RR_foot_imu_link">
+        <mu1>0.2</mu1>
+        <mu2>0.2</mu2>
+        <material>Gazebo/Red</material>
+    </gazebo>
     <!-- FL leg -->
     <gazebo reference="FL_hip">

File: robots/a1_imu_description/xacro/leg.xacro (robot description, xacro)
@@ -131,9 +131,4 @@
             </inertial>
         </link>
-        <joint name="${name}_foot_fixed" type="fixed">
-            <origin rpy="0 0 0" xyz="0 0 ${-(calf_length)}"/>
-            <parent link="${name}_calf"/>
-            <child link="${name}_foot"/>
-        </joint>
         <link name="${name}_foot">
             <visual>
@@ -166,9 +161,9 @@
             </inertial>
         </link>
-    <joint name="${name}_imu_joint" type="fixed">
-        <parent link="${name}_foot"/>
-        <child link="${name}_foot_imu_link"/>
-        <origin rpy="0 0 0" xyz="0 0 0"/>
-    </joint>
+        <joint name="${name}_foot_fixed" type="fixed">
+            <origin rpy="0 0 0" xyz="0 0 ${-(calf_length)}"/>
+            <parent link="${name}_calf"/>
+            <child link="${name}_foot"/>
+        </joint>
     <link name="${name}_foot_imu_link">
         <inertial>
@@ -187,8 +182,21 @@
             <origin rpy="0 0 0" xyz="0 0 0"/>
             <geometry>
-                <box size=".001 .001 .001"/>
+                <sphere radius=".0001"/>
             </geometry>
+                <surface>
+                <friction>
+                <ode>
+                    <mu>1.0</mu>
+                    <mu2>1.0</mu2>
+                </ode>
+                </friction>
+            </surface>
         </collision>
     </link>
+    <joint name="${name}_imu_joint" type="fixed">
+        <parent link="${name}_foot"/>
+        <child link="${name}_foot_imu_link"/>
+        <origin rpy="0 0 0" xyz="0 0 0"/>
+    </joint>
         <xacro:leg_transmission name="${name}"/>
     </xacro:macro>

File: robots/a1_imu_description/xacro/robot.xacro (robot description, xacro)
@@ -9,13 +9,4 @@
     <!-- Rollover Protection mode will add an additional stick on the top, use "true" or "false" to switch it. -->
     <xacro:property name="rolloverProtection" value="false"/>
-    <!-- Debug mode will hung up the robot, use "true" or "false" to switch it. -->
-    <xacro:if value="$(arg DEBUG)">
-        <link name="world"/>
-        <joint name="base_static_joint" type="fixed">
-            <origin rpy="0 0 0" xyz="0 0 0"/>
-            <parent link="world"/>
-            <child link="base"/>
-        </joint>
-    </xacro:if>
     <link name="base">
         <visual>

Commit message: fix force sensing bug

File: robots/a1_imu_description/urdf/a1_imu.urdf (robot description, URDF)
Before this commit: robot a1_imu_description, 27 links, 26 joints
Links:
- link FL_foot_imu_link: geometry 
- link FR_foot_imu_link: geometry 
- link RL_foot_imu_link: geometry 
- link RR_foot_imu_link: geometry 

File: robots/a1_imu_description/xacro/gazebo.xacro (robot description, xacro)
@@ -203,37 +203,38 @@
     </gazebo>
     <!-- Foot contacts. -->
-    <gazebo reference="FR_calf">
+    <gazebo reference="FR_foot">
         <sensor name="FR_foot_contact" type="contact">
-        <!-- <updateRate>100</updateRate> -->
+        <updateRate>100</updateRate>
         <plugin name="contactPlugin" filename="libunitreeFootContactPlugin.so"/>
         <contact>
-            <collision>FR_calf_fixed_joint_lump__FR_foot_collision_1</collision>
+            <collision>FR_foot_collision</collision>
         </contact>
         </sensor>
     </gazebo>
-    <gazebo reference="FL_calf">
+    <gazebo reference="FL_foot">
         <sensor name="FL_foot_contact" type="contact">
-        <!-- <updateRate>100</updateRate> -->
+        <updateRate>100</updateRate>
         <plugin name="contactPlugin" filename="libunitreeFootContactPlugin.so"/>
         <contact>
-            <collision>FL_calf_fixed_joint_lump__FL_foot_collision_1</collision>
+        <!-- this is from the Gazebo GUI -->
+            <collision>FL_foot_collision</collision>
         </contact>
         </sensor>
     </gazebo>
-    <gazebo reference="RR_calf">
+    <gazebo reference="RR_foot">
         <sensor name="RR_foot_contact" type="contact">
-        <!-- <updateRate>100</updateRate> -->
+        <updateRate>100</updateRate>
         <plugin name="contactPlugin" filename="libunitreeFootContactPlugin.so"/>
         <contact>
-            <collision>RR_calf_fixed_joint_lump__RR_foot_collision_1</collision>
+            <collision>RR_foot_collision</collision>
         </contact>
         </sensor>
     </gazebo>
-    <gazebo reference="RL_calf">
+    <gazebo reference="RL_foot">
         <sensor name="RL_foot_contact" type="contact">
-        <!-- <updateRate>100</updateRate> -->
+        <updateRate>100</updateRate>
         <plugin name="contactPlugin" filename="libunitreeFootContactPlugin.so"/>
         <contact>
-            <collision>RL_calf_fixed_joint_lump__RL_foot_collision_1</collision>
+            <collision>RL_foot_collision</collision>
         </contact>
         </sensor>

File: robots/a1_imu_description/xacro/leg.xacro (robot description, xacro)
@@ -172,5 +172,5 @@
             <inertia ixx="0.0001" ixy="0" ixz="0" iyy="0.0001" iyz="0" izz="0.0001"/>
         </inertial>
-        <visual>
+        <!-- <visual>
             <origin rpy="0 0 0" xyz="0 0 0"/>
             <geometry>
@@ -192,5 +192,5 @@
                 </friction>
             </surface>
-        </collision>
+        </collision> -->
     </link>
     <joint name="${name}_imu_joint" type="fixed">
